File: hw/RF_module.brd (EAGLE design)
At the start: 25 x 45 mm, 27 parts, among them J1 R2P_BUS-VERTICAL, J2 R2P_BUS-VERTICAL

Commit message: Fixed silkscreen
Parts:
- U$5: value ABRACON_ASD -> OSC; device r2p_ic:ABRACON_2.5X2 -> r2p_ic:XTAL_2.5X2
Other:
- board text added: "RF module v1.0 (2015/02)"
- board text removed: "R2P module v0.0 (YYYY/MM)"
Changed lines of the file:
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@@
 <wire x1="6.55" y1="8" x2="6.55" y2="8.8" width="0.2" layer="41"/>
 <wire x1="6.55" y1="8.8" x2="7.45" y2="8.8" width="0.2" layer="41"/>
-<text x="4" y="6" size="1.5" layer="200" rot="MR90">R2P module
-v0.0 (YYYY/MM)</text>
+<text x="4" y="6" size="1.5" layer="200" rot="MR90">RF module
+v1.0 (2015/02)</text>
 <text x="21" y="42.5" size="1" layer="48" font="vector" rot="R90" align="center">LINK</text>
 </plain>
@@
 </element>
 <element name="U$1" library="r2p_pcb" package="25X45" value="PCB_25X45" x="0" y="0" smashed="yes"/>
-<element name="U$5" library="r2p_ic" package="ABRACON_2.5X2" value="ABRACON_ASD" x="22.7" y="16" smashed="yes" rot="R180">
+<element name="U$5" library="r2p_ic" package="XTAL_2.5X2" value="OSC" x="22.7" y="16" smashed="yes" rot="R180">
 <attribute name="NAME" x="22.7" y="16" size="1" layer="25" font="vector" rot="R180" align="center"/>
 <attribute name="VALUE" x="24.95" y="18.75" size="1.27" layer="27" rot="R180"/>
